File: ESP32-Temp.kicad_pcb (KiCad board)
At the start: 4 copper layers, 30 parts, among them J1 USB_C_Receptacle_USB2.0, U1 ESP32-S3-WROOM-1-N4R2, U2 AP2112K-3.3, U3 CP2102N-Axx-xQFN28

Commit message: push
Parts:
- added C10: 1uf, Capacitor_SMD:C_0402_1005Metric, F.Cu at (45.3, 79.5)
- added C10: 1nF, Capacitor_SMD:C_01005_0402Metric, F.Cu at (48.8, 81.4)
- added C11: 1nF, Capacitor_SMD:C_01005_0402Metric, F.Cu at (52.8, 81.4)
- added C12: 1000uf 25v, Capacitor_THT:CP_Radial_D10.0mm_P5.00mm, F.Cu at (37.2, 113.8)
- added D10: WS2812B, LED_SMD:LED_WS2812B-2020_PLCC4_2.0x2.0mm, F.Cu at (62.2, 97.9)
- added D11: LED, LED_SMD:LED_0402_1005Metric, F.Cu at (30.7, 121.3)
- added D7: WS2812B, LED_SMD:LED_WS2812B-2020_PLCC4_2.0x2.0mm, F.Cu at (47.5, 110.2)
- added D8: WS2812B, LED_SMD:LED_WS2812B-2020_PLCC4_2.0x2.0mm, F.Cu at (58.1, 97.9)
- added D9: WS2812B, LED_SMD:LED_WS2812B-2020_PLCC4_2.0x2.0mm, F.Cu at (47.5, 113.7)
- added F1: 1A, Fuse:Fuse_0603_1608Metric, F.Cu at (35.7, 120.8)
- added J2: Program, Connector_PinHeader_2.54mm:PinHeader_1x02_P2.54mm_Vertical, F.Cu at (41.6, 80.8)
- added J3: 5V Signals, Connector_PinHeader_2.54mm:PinHeader_1x10_P2.54mm_Vertical, F.Cu at (27.9, 57.4)
- added J4: I2C LCD, Connector_PinHeader_2.54mm:PinHeader_1x04_P2.54mm_Vertical, F.Cu at (31.3, 110.3)
- added J5: I2C Temp, Connector_PinHeader_2.54mm:PinHeader_1x04_P2.54mm_Vertical, F.Cu at (53.7, 98.5)
- added J7: Power, TerminalBlock_Phoenix:TerminalBlock_Phoenix_MKDS-1,5-4-5.08_1x04_P5.08mm_Horizontal, F.Cu at (32.6, 102.4)
- added Q1: SS8050-G, SS8050-G:TRANS_SS8050-G, F.Cu at (62.0, 47.4)
- added Q2: SS8050-G, SS8050-G:TRANS_SS8050-G, F.Cu at (45.6, 50.0)
- added R12: 22K, Resistor_SMD:R_01005_0402Metric, F.Cu at (56.6, 77.4)
- added R13: 1k1, Resistor_SMD:R_0603_1608Metric, F.Cu at (27.6, 83.8)
- added R13: 22K, Resistor_SMD:R_01005_0402Metric, F.Cu at (44.6, 47.8)
- added R14: 2k2, Resistor_SMD:R_01005_0402Metric, F.Cu at (31.4, 70.4)
- added R15: 2k2, Resistor_SMD:R_01005_0402Metric, F.Cu at (43.8, 60.6)
- added R16: 422, Resistor_SMD:R_01005_0402Metric, F.Cu at (50.7, 109.2)
- added R17: 1k1, Resistor_SMD:R_0603_1608Metric, F.Cu at (58.0, 101.0)
- added SW1: SW, Jumper:SolderJumper-2_P1.3mm_Open_Pad1.0x1.5mm, F.Cu at (48.9, 78.4)
- added SW2: SW, Jumper:SolderJumper-2_P1.3mm_Open_Pad1.0x1.5mm, F.Cu at (53.3, 78.4)
- added TP1: TestPoint, Connector_PinHeader_2.54mm:PinHeader_1x01_P2.54mm_Vertical, F.Cu at (45.0, 57.4)
- added TP2: TestPoint, Connector_PinHeader_2.54mm:PinHeader_1x01_P2.54mm_Vertical, F.Cu at (54.3, 57.4)
- added TP3: TestPoint, Connector_PinHeader_2.54mm:PinHeader_1x01_P2.54mm_Vertical, F.Cu at (49.7, 57.4)
- added U4: 74HC245, Package_SO:SO-20_12.8x7.5mm_P1.27mm, F.Cu at (36.5, 62.3)
- R10, R11: footprint Resistor_SMD:R_0603_1608Metric -> Resistor_SMD:R_01005_0402Metric
- moved R10 5.51 mm to (47.8, 48.9), turned to -90 degrees
- moved R11 4.54 mm to (47.8, 51.2), turned to 90 degrees
Connections:
- C1 pad 2: USB_VDD -> GND
- C2 pad 2: USB_VDD -> GND
- C3 pad 2: USB_VDD -> GND
- C4 pad 1: Net-(C4-Pad1) -> USB_VDD
- C4 pad 2: USB_VDD -> GND
- C5 pad 1: USB_VDD -> GND
- C6 pad 1: USB_VDD -> GND
- C7 pad 1: Net-(C7-Pad1) -> /VBUS_REG
- C7 pad 2: USB_VDD -> GND
- C8 pad 2: USB_VDD -> GND
- C9 pad 2: USB_VDD -> GND
- D1 pad 1: Net-(C7-Pad1) -> VB_USB
- D2 pad 1: USB_VDD -> GND
- D5 pad 1: USB_VDD -> GND
- D6 pad 1: USB_VDD -> GND
- J1 pad A1: USB_VDD -> GND
- J1 pad A12: USB_VDD -> GND
- J1 pad B1: USB_VDD -> GND
- J1 pad B12: USB_VDD -> GND
- J1 pad S1: USB_VDD -> GND
- R1 pad 2: USB_VDD -> GND
- R2 pad 2: USB_VDD -> GND
- R3 pad 1: Net-(C7-Pad1) -> /VBUS_REG
- R4 pad 1: USB_VDD -> GND
- R5 pad 2: Net-(C4-Pad1) -> USB_VDD
- U1 pad 1: USB_VDD -> GND
- U1 pad 12: unconnected-(U1-Pad12) -> /a1
- U1 pad 17: unconnected-(U1-Pad17) -> /a2
- U1 pad 18: unconnected-(U1-Pad18) -> /a3
- U1 pad 19: unconnected-(U1-Pad19) -> /a4
- U1 pad 20: unconnected-(U1-Pad20) -> /a5
- U1 pad 21: unconnected-(U1-Pad21) -> /a6
- U1 pad 22: unconnected-(U1-Pad22) -> /a7
- U1 pad 27: unconnected-(U1-Pad27) -> BOOT
- U1 pad 4: unconnected-(U1-Pad4) -> SCL
- U1 pad 40: USB_VDD -> GND
- U1 pad 41_1: USB_VDD -> GND
- U1 pad 41_2: USB_VDD -> GND
- U1 pad 41_3: USB_VDD -> GND
- U1 pad 41_4: USB_VDD -> GND
- U1 pad 41_5: USB_VDD -> GND
- U1 pad 41_6: USB_VDD -> GND
- U1 pad 41_7: USB_VDD -> GND
- U1 pad 41_8: USB_VDD -> GND
- U1 pad 41_9: USB_VDD -> GND
- U1 pad 5: unconnected-(U1-Pad5) -> SDA
- U1 pad 7: unconnected-(U1-Pad7) -> /a0
- U2 pad 1: Net-(C7-Pad1) -> /VBUS_REG
- U2 pad 2: USB_VDD -> GND
- U3 pad 29: USB_VDD -> GND
- U3 pad 3: USB_VDD -> GND
- U3 pad 6: Net-(C4-Pad1) -> USB_VDD
Routing:
- net USB_VDD: track 20.1 -> 0.00 mm, vias 2 -> 0
- net GND: track 0.00 -> 20.1 mm, vias 0 -> 2
- net BOOT: track 0.00 -> 2.39 mm
- net DTR: track 0.00 -> 2.34 mm
- net Net-(Q2-Pad1): track 0.00 -> 1.82 mm

Commit message: JLCPCB Order
Parts:
- removed the C10 at (45.3, 79.5)
- removed the C10 at (48.8, 81.4)
- removed J2: Program, Connector_PinHeader_2.54mm:PinHeader_1x02_P2.54mm_Vertical
- removed the R13 at (27.6, 83.8)
- removed the R13 at (44.6, 47.8)
- added C10: 1000uf 25v, Capacitor_THT:CP_Radial_D10.0mm_P5.00mm, F.Cu at (29.8, 46.2)
- added J6: PowerSelector, Connector_PinHeader_2.54mm:PinHeader_2x03_P2.54mm_Vertical, F.Cu at (17.4, 43.7)
- added J_5V1: Ext_Power_IN, Connector_JST:JST_EH_B4B-EH-A_1x04_P2.50mm_Vertical, F.Cu at (26.8, 55.1)
- added J_5V2: Ext_Power_OUT, Connector_JST:JST_EH_B4B-EH-A_1x04_P2.50mm_Vertical, F.Cu at (40.8, 55.1)
- added J_I2C1: I2C Temp, Connector_PinHeader_2.54mm:PinHeader_1x04_P2.54mm_Vertical, F.Cu at (70.4, 23.2)
- added J_LCD1: I2C LCD, Connector_PinHeader_2.54mm:PinHeader_1x04_P2.54mm_Vertical, F.Cu at (74.2, 23.2)
- added R13: 422, Resistor_THT:R_Axial_DIN0207_L6.3mm_D2.5mm_P2.54mm_Vertical, F.Cu at (47.0, 49.3)
- added R18: 22K, Resistor_SMD:R_01005_0402Metric, F.Cu at (62.5, 30.2)
- added R19: 100k, Resistor_SMD:R_01005_0402Metric, F.Cu at (44.1, 25.0)
- added R20: 2k2, Resistor_SMD:R_01005_0402Metric, F.Cu at (61.0, 31.7)
- added R21: 2k2, Resistor_SMD:R_01005_0402Metric, F.Cu at (63.8, 31.7)
- added R22: 422, Resistor_THT:R_Axial_DIN0207_L6.3mm_D2.5mm_P2.54mm_Vertical, F.Cu at (57.4, 24.6)
- added R23: 422, Resistor_THT:R_Axial_DIN0207_L6.3mm_D2.5mm_P2.54mm_Vertical, F.Cu at (60.5, 24.6)
- added R24: 422, Resistor_THT:R_Axial_DIN0207_L6.3mm_D2.5mm_P2.54mm_Vertical, F.Cu at (63.5, 24.6)
- added R25: 422, Resistor_THT:R_Axial_DIN0207_L6.3mm_D2.5mm_P2.54mm_Vertical, F.Cu at (66.5, 24.6)
- added TPG1: TestPoint, TestPoint:TestPoint_THTPad_1.0x1.0mm_Drill0.5mm, F.Cu at (55.9, 28.2)
- C1, C6: value 0.1uf -> 1uf
- C11: value 1nF -> 1uf; footprint Capacitor_SMD:C_01005_0402Metric -> Capacitor_SMD:C_0402_1005Metric
- C12: value 1000uf 25v -> 1nF; footprint Capacitor_THT:CP_Radial_D10.0mm_P5.00mm -> Capacitor_SMD:C_01005_0402Metric
- C2: value 1uf -> 0.1uf
- C3: value 10uf -> 0.1uf
- C9: value 1uf -> 10uf
- D1: value MBR0540 -> SP0503BAHTG; footprint Diode_SMD:D_SOD-123 -> SP0503BAHTG:SOT143
- D10, D7, D8, D9: value WS2812B -> LED; footprint LED_SMD:LED_WS2812B-2020_PLCC4_2.0x2.0mm -> LED_SMD:LED_0402_1005Metric
- D2: value SP0503BAHTG -> MBR0540; footprint SP0503BAHTG:SOT143 -> Diode_SMD:D_SOD-123
- D3, D4, D5, D6: value LED -> WS2812B; footprint LED_SMD:LED_0402_1005Metric -> LED_SMD:LED_WS2812B-2020_PLCC4_2.0x2.0mm
- F1: footprint Fuse:Fuse_0603_1608Metric -> Capacitor_THT:C_Disc_D5.0mm_W2.5mm_P2.50mm
- J3: value 5V Signals -> IO_2; footprint Connector_PinHeader_2.54mm:PinHeader_1x10_P2.54mm_Vertical -> Connector_PinHeader_1.27mm:PinHeader_1x09_P1.27mm_Vertical
- J4: value I2C LCD -> LED_MATRIX; footprint Connector_PinHeader_2.54mm:PinHeader_1x04_P2.54mm_Vertical -> Connector_PinHeader_2.54mm:PinHeader_1x03_P2.54mm_Vertical
- J5: value I2C Temp -> Program; footprint Connector_PinHeader_2.54mm:PinHeader_1x04_P2.54mm_Vertical -> Connector_PinHeader_2.54mm:PinHeader_1x02_P2.54mm_Vertical
- J7: value Power -> Conn_01x09_Pin; footprint TerminalBlock_Phoenix:TerminalBlock_Phoenix_MKDS-1,5-4-5.08_1x04_P5.08mm_Horizontal -> Connector_PinHeader_2.54mm:PinHeader_1x09_P2.54mm_Vertical
- R10, R11: value 100k -> 1k1; footprint Resistor_SMD:R_01005_0402Metric -> Resistor_SMD:R_0603_1608Metric
- R12: value 22K -> 1k1; footprint Resistor_SMD:R_01005_0402Metric -> Resistor_SMD:R_0603_1608Metric
- R14, R15: value 2k2 -> 422; footprint Resistor_SMD:R_01005_0402Metric -> Resistor_THT:R_Axial_DIN0207_L6.3mm_D2.5mm_P2.54mm_Vertical
- R16: footprint Resistor_SMD:R_01005_0402Metric -> Resistor_THT:R_Axial_DIN0207_L6.3mm_D2.5mm_P2.54mm_Vertical
- R17: value 1k1 -> 100k; footprint Resistor_SMD:R_0603_1608Metric -> Resistor_SMD:R_01005_0402Metric
- R3, R4: value 100k -> 1k1
- R5, R6: value 1k1 -> 100k
- R7: value 1k1 -> 422; footprint Resistor_SMD:R_0603_1608Metric -> Resistor_SMD:R_01005_0402Metric
- SW1: value SW -> EN_SW
- SW2: value SW -> BOOT_SW
- TP1, TP2, TP3: footprint Connector_PinHeader_2.54mm:PinHeader_1x01_P2.54mm_Vertical -> TestPoint:TestPoint_THTPad_1.0x1.0mm_Drill0.5mm
- U2: value AP2112K-3.3 -> 74HC245; footprint Package_TO_SOT_SMD:SOT-23-5 -> Package_SO:SOIC-20W_7.5x12.8mm_P1.27mm
- U4: value 74HC245 -> AP2112K-3.3; footprint Package_SO:SO-20_12.8x7.5mm_P1.27mm -> Package_TO_SOT_SMD:SOT-23-5
- moved J7 93.6 mm to (74.2, 18.6), turned to -90 degrees
- moved C4 89.7 mm to (25.4, 25.9), turned to 90 degrees
- moved D11 89.3 mm to (30.7, 32.0), turned to -90 degrees
- moved D10 89.2 mm to (17.5, 20.7), turned to 180 degrees
- moved R7 85.6 mm to (37.5, 20.3)
- moved R16 84.7 mm to (54.4, 24.6), turned to 90 degrees
- moved C9 84.5 mm to (26.7, 36.1), turned to 180 degrees
- moved F1 84.2 mm to (17.5, 38.6), turned to 90 degrees
- moved R6 83.8 mm to (20.8, 39.4)
- moved D4 82.6 mm to (41.5, 18.5)
- moved D7 82.5 mm to (38.5, 28.2)
- moved D3 81.9 mm to (38.4, 18.5)
- moved R5 81.8 mm to (23.6, 35.2), turned to 90 degrees
- moved C8 81.5 mm to (20.8, 40.9)
- moved D9 79.4 mm to (30.0, 36.3)
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Connections:
- C1 pad 1: 3v3 -> VBUS
- C11 pad 1: BOOT -> EN
- C12 pad 1: EXT_5V -> BOOT
- C2 pad 1: 3v3 -> GND
- C2 pad 2: GND -> VBUS
- C3 pad 1: 3v3 -> GND
- C3 pad 2: GND -> VBUS
- C5 pad 1: GND -> 3v3
- C5 pad 2: VBUS -> GND
- C6 pad 1: GND -> 3v3
- C6 pad 2: VBUS -> GND
- C7 pad 1: /VBUS_REG -> 3v3
- C8 pad 1: 3v3 -> /VBUS_REG
- C9 pad 1: VBUS -> 3v3
- D1 pad 1: VB_USB -> GND
- D10 pad 1: /VBUS_REG -> GND
- D10 pad 2: unconnected-(D10-Pad2) -> Net-(D10-A)
- D11 pad 2: Net-(D11-Pad2) -> Net-(D11-A)
- D2 pad 1: GND -> VB_USB
- D3 pad 1: TXT -> /VBUS_REG
- D3 pad 2: Net-(D3-Pad2) -> Net-(D3-DOUT)
- D4 pad 1: RXT -> /VBUS_REG
- D4 pad 2: Net-(D4-Pad2) -> Net-(D4-DOUT)
- D5 pad 1: GND -> /VBUS_REG
- D5 pad 2: Net-(D5-Pad2) -> Net-(D5-DOUT)
- D6 pad 1: GND -> /VBUS_REG
- D6 pad 2: Net-(D6-Pad2) -> unconnected-(D6-DOUT-Pad2)
- D7 pad 1: /VBUS_REG -> TXT
- D7 pad 2: Net-(D7-Pad2) -> Net-(D7-A)
- D8 pad 1: /VBUS_REG -> RXT
- D8 pad 2: Net-(D8-Pad2) -> Net-(D8-A)
- D9 pad 1: /VBUS_REG -> GND
- D9 pad 2: Net-(D10-Pad4) -> Net-(D9-A)
- J3 pad 1: GND -> /IO48
- J3 pad 2: /b7 -> /IO47
- J3 pad 3: /b6 -> /IO46
- J3 pad 4: /b5 -> /IO45
- J3 pad 5: /b4 -> /IO42
- J3 pad 6: /b3 -> /IO41
- J3 pad 7: /b2 -> /IO40
- J3 pad 8: /b1 -> /IO39
- J3 pad 9: /b0 -> /IO38
- J4 pad 1: SDA -> Net-(J4-Pin_1)
- J4 pad 2: SCL -> GND
- J4 pad 3: 3v3 -> /VBUS_REG
- J5 pad 1: SDA -> USB_RXD
- J5 pad 2: SCL -> USB_TXD
- J7 pad 2: EXT_5V -> Net-(J7-Pin_2)
- J7 pad 3: (no net) -> Net-(J7-Pin_3)
- J7 pad 4: (no net) -> Net-(J7-Pin_4)
- R10 pad 1: DTR -> Net-(D9-A)
- R10 pad 2: Net-(Q1-Pad1) -> 3v3
- R11 pad 1: RTS -> Net-(D10-A)
- R11 pad 2: Net-(Q2-Pad1) -> VBUS
- R12 pad 1: 3v3 -> Net-(D11-A)
- R12 pad 2: EN -> /VBUS_REG
- R14 pad 1: 3v3 -> /b1
- R14 pad 2: SDA -> Net-(J7-Pin_8)
- R15 pad 1: 3v3 -> /b2
- R15 pad 2: SCL -> Net-(J7-Pin_7)
- R16 pad 1: /b7 -> /b3
- R16 pad 2: Net-(D7-Pad4) -> Net-(J7-Pin_6)
- R17 pad 1: Net-(D11-Pad2) -> DTR
- R17 pad 2: /VBUS_REG -> Net-(Q1-Pad1)
- R3 pad 1: /VBUS_REG -> Net-(U3-~{RST})
- R3 pad 2: Net-(R3-Pad2) -> USB_VDD
- R4 pad 1: GND -> Net-(U2-A->B)
- R4 pad 2: VBUS -> /VBUS_REG
- R5 pad 1: Net-(R5-Pad1) -> GND
- R5 pad 2: USB_VDD -> VBUS
- R6 pad 1: Net-(D3-Pad2) -> /VBUS_REG
- R6 pad 2: USB_VDD -> Net-(U4-EN)
- R7 pad 1: Net-(D4-Pad2) -> /b7
- R7 pad 2: USB_VDD -> Net-(D3-DIN)
- R8 pad 1: Net-(D5-Pad2) -> Net-(D7-A)
- R8 pad 2: 3v3 -> USB_VDD
- R9 pad 1: Net-(D6-Pad2) -> Net-(D8-A)
- R9 pad 2: VBUS -> USB_VDD
- U1 pad 11: unconnected-(U1-Pad11) -> /IO18
- U1 pad 13: unconnected-(U1-Pad13) -> /IO19
- U1 pad 14: unconnected-(U1-Pad14) -> /IO20
- U1 pad 16: unconnected-(U1-Pad16) -> /IO46
- U1 pad 23: unconnected-(U1-Pad23) -> /IO21
- U1 pad 24: unconnected-(U1-Pad24) -> /IO47
- U1 pad 25: unconnected-(U1-Pad25) -> /IO48
- U1 pad 26: unconnected-(U1-Pad26) -> /IO45
- U1 pad 28: unconnected-(U1-Pad28) -> /IO35
- U1 pad 29: unconnected-(U1-Pad29) -> /IO36
- U1 pad 30: unconnected-(U1-Pad30) -> /IO37
- U1 pad 31: unconnected-(U1-Pad31) -> /IO38
- U1 pad 32: unconnected-(U1-Pad32) -> /IO39
- U1 pad 33: unconnected-(U1-Pad33) -> /IO40
- U1 pad 34: unconnected-(U1-Pad34) -> /IO41
- U1 pad 35: unconnected-(U1-Pad35) -> /IO42
- U1 pad 8: unconnected-(U1-Pad8) -> /IO15
- U1 pad 9: unconnected-(U1-Pad9) -> /IO16
- U2 pad 1: /VBUS_REG -> Net-(U2-A->B)
- U2 pad 2: GND -> /a0
- U2 pad 3: Net-(R3-Pad2) -> /a1
- U2 pad 4: unconnected-(U2-Pad4) -> /a2
- U2 pad 5: 3v3 -> /a3
- U3 pad 9: Net-(R5-Pad1) -> Net-(U3-~{RST})
- U4 pad 1: Net-(R13-Pad1) -> /VBUS_REG
- U4 pad 2: /a0 -> GND
- U4 pad 3: /a1 -> Net-(U4-EN)
- U4 pad 4: /a2 -> unconnected-(U4-NC-Pad4)
- U4 pad 5: /a3 -> 3v3
Routing:
- net 3v3: track 0.00 -> 92.5 mm
- net USB_RXD: track 0.00 -> 68.9 mm, vias 0 -> 1
- net USB_TXD: track 0.00 -> 65.3 mm, vias 0 -> 1
- net EN: track 0.00 -> 62.3 mm
- net /b7: track 0.00 -> 53.2 mm
- net BOOT: track 2.39 -> 54.7 mm
- net VBUS: track 8.17 -> 50.9 mm
- net Net-(U3-~{RST}): track 0.00 -> 39.4 mm
- net USB_VDD: track 0.00 -> 38.7 mm
- net /a0: track 0.00 -> 29.2 mm
- net /IO46: track 0.00 -> 25.9 mm
- net GND: track 20.1 -> 43.7 mm, vias 2 -> 14
- net /b0: track 0.00 -> 22.9 mm
- net /b6: track 0.00 -> 22.1 mm
- net /IO48: track 0.00 -> 21.3 mm, vias 0 -> 1
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- added copper zone on In2.Cu, net /VBUS_REG
- added copper zone on F.Cu, net EXT_5V
- added copper zone on B.Cu, net GND
- added copper zone on F.Cu, net GND
- added copper zone on In1.Cu, net GND
Other:
- board outline added: 62.2 x 43.3 mm
- board text added: "+"
- board text added: "+ - D"
- board text added: "-"
- board text added: "3v3"
- board text added: "Boot"
- board text added: "EN"
- board text added: "ESP Board v1 - 03/23"
- board text added: "GND"
- board text added: "GPIOs"
- board text added: "Gnd"
- board text added: "Pratap Karonde"
- board text added: "Pwr In"
- board text added: "Pwr Out"
- board text added: "SCL"
- board text added: "SDA"
- board text added: "TTL Out"
- board text added: "Tx Rx"
- board text added: "USB VDD"
- board text added: "VBUS"
- board text added: "VSEL"

Commit message: JLCPCB Order again
Parts:
- C12: footprint Capacitor_SMD:C_01005_0402Metric -> Capacitor_SMD:C_0402_1005Metric
- R1, R17, R18, R19, R2, R20, R21: footprint Resistor_SMD:R_01005_0402Metric -> Resistor_SMD:R_0402_1005Metric
- R13, R14, R15, R16, R22, R23, R24, R25: footprint Resistor_THT:R_Axial_DIN0207_L6.3mm_D2.5mm_P2.54mm_Vertical -> Resistor_THT:R_Axial_DIN0204_L3.6mm_D1.6mm_P5.08mm_Horizontal
- R7: footprint Resistor_SMD:R_01005_0402Metric -> Resistor_THT:R_Axial_DIN0204_L3.6mm_D1.6mm_P5.08mm_Horizontal
- moved TPG1 22.3 mm to (75.6, 17.7)
- moved SW1 21.5 mm to (41.3, 23.4), turned to 90 degrees
- moved R19 6.65 mm to (50.7, 26.0)
- moved R14 6.43 mm to (54.4, 26.7)
- moved Q2 6.13 mm to (50.2, 23.5)
- moved R17 6.12 mm to (46.4, 26.0)
- moved R13 6.02 mm to (41.0, 48.8), turned to 0 degrees
- moved TP3 5.97 mm to (32.9, 34.6)
- moved Q1 5.92 mm to (46.5, 23.5)
- moved R7 5.87 mm to (37.0, 26.2), turned to 90 degrees
- moved C8 5.80 mm to (23.0, 35.5), turned to 90 degrees
- moved R15 5.59 mm to (56.5, 26.7)
- moved R16 4.77 mm to (58.7, 26.7)
- moved C12 4.53 mm to (48.5, 49.0), turned to 90 degrees
- moved R22 3.99 mm to (60.8, 26.7)
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Connections:
- U1 pad 11: /IO18 -> unconnected-(U1-IO18-Pad11)
- U1 pad 13: /IO19 -> unconnected-(U1-IO19-Pad13)
- U1 pad 14: /IO20 -> unconnected-(U1-IO20-Pad14)
- U1 pad 23: /IO21 -> unconnected-(U1-IO21-Pad23)
- U1 pad 28: /IO35 -> unconnected-(U1-IO35-Pad28)
- U1 pad 29: /IO36 -> unconnected-(U1-IO36-Pad29)
- U1 pad 30: /IO37 -> unconnected-(U1-IO37-Pad30)
- U1 pad 8: /IO15 -> unconnected-(U1-IO15-Pad8)
- U1 pad 9: /IO16 -> unconnected-(U1-IO16-Pad9)
Routing:
- net /VBUS_REG: track 18.2 -> 106.7 mm, vias 8 -> 0
- net 3v3: track 92.5 -> 27.2 mm, vias 0 -> 1
- net GND: track 43.7 -> 80.5 mm, vias 14 -> 48
- net BOOT: track 54.7 -> 91.4 mm
- net Net-(U3-~{RST}): track 39.4 -> 18.8 mm, vias 0 -> 2
- net USB_D+: track 18.1 -> 36.1 mm, vias 2 -> 0
- net EN: track 62.3 -> 44.8 mm
- net SDA: track 19.7 -> 29.9 mm, vias 1 -> 0
- net USB_VDD: track 38.7 -> 47.9 mm, vias 0 -> 2
- net DTR: track 17.9 -> 26.6 mm, vias 0 -> 2
- net USB_D-: track 16.7 -> 23.4 mm, vias 0 -> 2
- net Net-(J7-Pin_8): track 9.66 -> 3.21 mm
- net /b0: track 22.9 -> 16.7 mm
- net Net-(J7-Pin_7): track 9.07 -> 3.05 mm
- net RTS: track 13.7 -> 19.7 mm
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- added copper zone on In2.Cu, net 3v3
- removed copper zone on In2.Cu, net /VBUS_REG
Other:
- board text added: "12"
- board text added: "17"
- board text added: "18"
- board text added: "19"
- board text added: "20"
- board text added: "21"
- board text added: "22"
- board text added: "38"
- board text added: "39"
- board text added: "40"
- board text added: "41"
- board text added: "42"
- board text added: "45"
- board text added: "46"
- board text added: "47"
- board text added: "48"
- board text added: "5V"
- board text added: "ESP32-S3-WROOM-1-N4R2"
- board text added: "Ext-5V"
- board text added: "Pratap Karonde March 2023"
- board text added: "RX"
- board text added: "Rx"
- board text added: "TX"
- board text added: "Tx"
- board text added: "VBR"
- board text added: "VBus"
- board text added: "WS2812"
