File: ESP32-Temp.kicad_sch (KiCad schematic)
At the start: 38 parts, among them J1 USB_C_Receptacle_USB2.0, Q1 SS8050-G, Q2 SS8050-G, SW1 SW, SW2 SW, U1 ESP32-S3-WROOM-1-N4R2, U2 AP2112K-3.3, U3 CP2102N-Axx-xQFN28

Commit message: push
Parts:
- removed C10: 1nF, Capacitor_SMD:C_01005_0402Metric, symbol Device:C
- removed R13: 22K, Resistor_SMD:R_01005_0402Metric, symbol Device:R
- added C10: 1uf, Capacitor_SMD:C_0402_1005Metric, symbol Device:C_Small
- added C12: 1000uf 25v, Capacitor_THT:CP_Radial_D10.0mm_P5.00mm, symbol Device:C_Polarized
- added D10, D7, D8, D9: WS2812B, LED_SMD:LED_WS2812B-2020_PLCC4_2.0x2.0mm, symbol LED:WS2812B
- added D11: LED, LED_SMD:LED_0402_1005Metric, symbol Device:LED
- added F1: 1A, Fuse:Fuse_0603_1608Metric, symbol Device:Polyfuse
- added J2: Program, Connector_PinHeader_2.54mm:PinHeader_1x02_P2.54mm_Vertical, symbol Connector:Conn_01x02_Male
- added J3: 5V Signals, Connector_PinHeader_2.54mm:PinHeader_1x10_P2.54mm_Vertical, symbol Connector:Conn_01x10_Male
- added J4: I2C LCD, Connector_PinHeader_2.54mm:PinHeader_1x04_P2.54mm_Vertical, symbol Connector:Conn_01x04_Female
- added J5: I2C Temp, Connector_PinHeader_2.54mm:PinHeader_1x04_P2.54mm_Vertical, symbol Connector:Conn_01x04_Female
- added J6: PowerSelector, symbol Connector:Conn_01x03_Female
- added J?: Ext_Power, TerminalBlock_Phoenix:TerminalBlock_Phoenix_MKDS-1,5-4-5.08_1x04_P5.08mm_Horizontal, symbol Connector_Generic:Conn_01x04
- added R13, R17: 1k1, Resistor_SMD:R_0603_1608Metric, symbol Device:R_Small
- added R14, R15: 2k2, Resistor_SMD:R_01005_0402Metric, symbol Device:R
- added R16, R? (x4): 422, Resistor_SMD:R_01005_0402Metric, symbol Device:R
- added TP1, TP2, TP3: TestPoint, Connector_PinHeader_2.54mm:PinHeader_1x01_P2.54mm_Vertical, symbol Connector:TestPoint
- added U4: 74HC245, Package_SO:SO-20_12.8x7.5mm_P1.27mm, symbol 74xx:74HC245
- R10, R11: footprint Resistor_SMD:R_0603_1608Metric -> Resistor_SMD:R_01005_0402Metric; LCSC C319969 -> C25741
Connections:
- net 3v3: now also J4.3 (Pin_3), J5.4 (Pin_4), R14.1, R15.1, TP3.1
- net EN: now also C10.1
- net GND: now also C10.2, C12.2, D10.3 (VSS), D11.1 (K), D7.3 (VSS), D8.3 (VSS), D9.3 (VSS), J3.1 (Pin_1), J4.4 (Pin_4), J5.3 (Pin_3), J?.1 (Pin_1), J?.2 (Pin_2), U4.10 (GND), U4.19 (CE); no longer R6.2, R7.2
- net USB_RXD: now also J2.1 (Pin_1)
- net USB_TXD: now also J2.2 (Pin_2)
- net VBUS: now also TP1.1
- net a1: now reaches U1.12 (IO8)
- net a1: now also U4.3 (A1)
- net a2: now reaches U1.17 (IO9)
- net a2: now also U4.4 (A2)
- net a3: now reaches U1.18 (IO10)
- net a3: now also U4.5 (A3)
- net a4: now reaches U1.19 (IO11)
- net a4: now also U4.6 (A4)
- net a5: now reaches U1.20 (IO12)
- net a5: now also U4.7 (A5)
- net a6: now reaches U1.21 (IO13)
- net a6: now also U4.8 (A6)
- net a7: now reaches U1.22 (IO14)
- net a7: now also U4.9 (A7)
- net SCL: now reaches U1.4 (IO4)
- net SCL: now also J4.2 (Pin_2), J5.2 (Pin_2), R15.2
- net SDA: now reaches U1.5 (IO5)
- net SDA: now also J4.1 (Pin_1), J5.1 (Pin_1), R14.2
- net a0: now reaches U1.7 (IO7)
- net a0: now also U4.2 (A0)
- net VBUS_REG: now reaches C7.1, R3.1, U2.1 (VIN)
- net VBUS_REG: now also D10.1 (VDD), D7.1 (VDD), D8.1 (VDD), D9.1 (VDD), F1.2, R13.2, R17.2, U4.20 (VCC); no longer D1.1 (K)
- net USB_VDD: now reaches C4.1, R5.2, U3.6 (VDD)
- net USB_VDD: now also R6.2, R7.2, TP2.1
- new net: J3.8 (Pin_8), R?.2
- new net: D7.4 (DIN), R16.2
- new net: J3.6 (Pin_6), R?.2
- new net: J3.7 (Pin_7), R?.2
- new net: J3.9 (Pin_9), R?.2
- new net: D7.2 (DOUT), D8.4 (DIN)
- new net: D8.2 (DOUT), D9.4 (DIN)
- new net: R13.1, U4.1 (A->B)
- new net: D10.4 (DIN), D9.2 (DOUT)
- new net: D11.2 (A), R17.1
- new net EXT_5V: C12.1, J3.10 (Pin_10), J6.3 (Pin_3), J?.3 (Pin_3), J?.4 (Pin_4)
- new net VB_USB: D1.1 (K), J6.1 (Pin_1)
- new net V_SEL: F1.1, J6.2 (Pin_2)
- new net b0: R?.1, U4.18 (B0)
- new net b1: R?.1, U4.17 (B1)
- new net b2: R?.1, U4.16 (B2)
- new net b3: R?.1, U4.15 (B3)
- new net b4: J3.5 (Pin_5), U4.14 (B4)
- new net b5: J3.4 (Pin_4), U4.13 (B5)
- new net b6: J3.3 (Pin_3), U4.12 (B6)
- new net b7: J3.2 (Pin_2), R16.1, U4.11 (B7)
- no-connect marks 16 -> 18
Other:
- note added: "Auto Program DTR RTS-->EN IO0 1 1 1 1 0 0 1 1 1 0 0 1 0 1 1 0 (Program)"
- note added: "Close this jumper to power circuit from external source !! Remove USB Cable First"
- note added: "I2C Pullup"
- moved on the sheet: C4, C5, C6, C7, C8, C9, D1, D2, R3, R4, R5, U2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

Commit message: JLCPCB Order
Parts:
- removed J3: 5V Signals, Connector_PinHeader_2.54mm:PinHeader_1x10_P2.54mm_Vertical, symbol Connector:Conn_01x10_Male
- removed J6: PowerSelector, symbol Connector:Conn_01x03_Female
- added J3: IO_2, Connector_PinHeader_1.27mm:PinHeader_1x09_P1.27mm_Vertical, symbol Connector:Conn_01x09_Male
- added J4: LED_MATRIX, Connector_PinHeader_2.54mm:PinHeader_1x03_P2.54mm_Vertical, symbol Connector:Conn_01x03_Pin
- added J6: PowerSelector, Connector_PinHeader_2.54mm:PinHeader_2x03_P2.54mm_Vertical, symbol Connector_Generic:Conn_02x03_Top_Bottom
- added J7: Conn_01x09_Pin, Connector_PinHeader_2.54mm:PinHeader_1x09_P2.54mm_Vertical, symbol Connector:Conn_01x09_Pin
- added J_5V2: Ext_Power_OUT, Connector_JST:JST_EH_B4B-EH-A_1x04_P2.50mm_Vertical, symbol Connector_Generic:Conn_01x04
- added R22, R23, R24, R25: 422, Resistor_THT:R_Axial_DIN0207_L6.3mm_D2.5mm_P2.54mm_Vertical, symbol Device:R
- added TPG1: TestPoint, TestPoint:TestPoint_THTPad_1.0x1.0mm_Drill0.5mm, symbol Connector:TestPoint
- F1: footprint Fuse:Fuse_0603_1608Metric -> Capacitor_THT:C_Disc_D5.0mm_W2.5mm_P2.50mm; LCSC C122964 -> (none)
- J_5V1: renamed from J?; value Ext_Power -> Ext_Power_IN; footprint TerminalBlock_Phoenix:TerminalBlock_Phoenix_MKDS-1,5-4-5.08_1x04_P5.08mm_Horizontal -> Connector_JST:JST_EH_B4B-EH-A_1x04_P2.50mm_Vertical
- R13, R14, R15, R16: renamed from R?; footprint Resistor_SMD:R_01005_0402Metric -> Resistor_THT:R_Axial_DIN0207_L6.3mm_D2.5mm_P2.54mm_Vertical
- SW1: value SW -> EN_SW
- SW2: value SW -> BOOT_SW
- TP1, TP2, TP3: footprint Connector_PinHeader_2.54mm:PinHeader_1x01_P2.54mm_Vertical -> TestPoint:TestPoint_THTPad_1.0x1.0mm_Drill0.5mm
- U2: renamed from U4; footprint Package_SO:SO-20_12.8x7.5mm_P1.27mm -> Package_SO:SOIC-20W_7.5x12.8mm_P1.27mm
- renumbered C9 to C1, C12 to C10, C10 to C11, C11 to C12, C5 to C2, C6 to C3, C1 to C5, C2 to C6, C3 to C7, C7 to C8, C8 to C9, D2 to D1, D6 to D10, D1 to D2, D7 to D3, D8 to D4, D9 to D5, D10 to D6, D3 to D7, D4 to D8, D5 to D9, J2 to J5, J5 to J_I2C1, J4 to J_LCD1, R8 to R10, R9 to R11, R17 to R12, R10 to R17, R12 to R18, R11 to R19, R14 to R20, R15 to R21, R5 to R3, R13 to R4, R4 to R5, R3 to R6, R16 to R7, R6 to R8, R7 to R9, U2 to U4
Connections:
- net 3v3: now also J_LCD1.4 (Pin_4); no longer J_LCD1.3 (Pin_3)
- net EXT_5V: now also J_5V1.1 (Pin_1), J_5V1.2 (Pin_2), J6.5 (Pin_5), J6.6 (Pin_6), J_5V2.3 (Pin_3), J_5V2.4 (Pin_4); no longer J_5V1.3 (Pin_3), J_5V1.4 (Pin_4)
- net GND: now also J_5V1.3 (Pin_3), J_5V1.4 (Pin_4), J_LCD1.3 (Pin_3), J4.2 (Pin_2), J7.1 (Pin_1), J_5V2.1 (Pin_1), J_5V2.2 (Pin_2), TPG1.1; no longer J_5V1.1 (Pin_1), J_5V1.2 (Pin_2), J_LCD1.4 (Pin_4)
- net VBUS_REG: now also J4.3 (Pin_3), J7.9 (Pin_9)
- net VB_USB: now also J6.1 (Pin_1), J6.2 (Pin_2)
- net V_SEL: now also J6.3 (Pin_3), J6.4 (Pin_4)
- net b4: now also R22.1
- net b5: now also R23.1
- net b6: now also R24.1
- net b7: now also R25.1
- net at R14.2: now also J7.8 (Pin_8)
- net IO18: now reaches U1.11 (IO18)
- net IO19: now reaches U1.13 (IO19)
- net IO20: now reaches U1.14 (IO20)
- net IO46: now reaches U1.16 (IO46)
- net IO46: now also J3.3 (Pin_3)
- net IO21: now reaches U1.23 (IO21)
- net IO47: now reaches U1.24 (IO47)
- net IO47: now also J3.2 (Pin_2)
- net IO48: now reaches U1.25 (IO48)
- net IO48: now also J3.1 (Pin_1)
- net IO45: now reaches U1.26 (IO45)
- net IO45: now also J3.4 (Pin_4)
- net IO35: now reaches U1.28 (IO35)
- net IO36: now reaches U1.29 (IO36)
- net IO37: now reaches U1.30 (IO37)
- net IO38: now reaches U1.31 (IO38)
- net IO38: now also J3.9 (Pin_9)
- net IO39: now reaches U1.32 (IO39)
- net IO39: now also J3.8 (Pin_8)
- net IO40: now reaches U1.33 (IO40)
- net IO40: now also J3.7 (Pin_7)
- net IO41: now reaches U1.34 (IO41)
- net IO41: now also J3.6 (Pin_6)
- net IO42: now reaches U1.35 (IO42)
- net IO42: now also J3.5 (Pin_5)
- net IO15: now reaches U1.8 (IO15)
- net IO16: now reaches U1.9 (IO16)
- net at R16.2: now also J7.6 (Pin_6)
- net at R15.2: now also J7.7 (Pin_7)
- net at R13.2: now also J4.1 (Pin_1)
- new net: J7.4 (Pin_4), R23.2
- new net: J7.3 (Pin_3), R24.2
- new net: J7.2 (Pin_2), R25.2
- new net: J7.5 (Pin_5), R22.2
- no-connect marks 18 -> 22
Other:
- moved on the sheet: C1, C10, C11, C12, C2, C3, C4, C5, C6, C7, D1, D10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

Commit message: JLCPCB Order again
Parts:
- C12: footprint Capacitor_SMD:C_01005_0402Metric -> Capacitor_SMD:C_0402_1005Metric
- R1, R17, R18, R19, R2, R20, R21: footprint Resistor_SMD:R_01005_0402Metric -> Resistor_SMD:R_0402_1005Metric
- R13: footprint Resistor_THT:R_Axial_DIN0207_L6.3mm_D2.5mm_P2.54mm_Vertical -> R_Axial_DIN0204_L3.6mm_D1.6mm_P5.08mm_Horizontal; LCSC C11702 -> (none)
- R14, R15, R16, R22, R23, R24, R25: footprint Resistor_THT:R_Axial_DIN0207_L6.3mm_D2.5mm_P2.54mm_Vertical -> Resistor_THT:R_Axial_DIN0204_L3.6mm_D1.6mm_P5.08mm_Horizontal; LCSC C11702 -> (none)
- R7: footprint Resistor_SMD:R_01005_0402Metric -> Resistor_THT:R_Axial_DIN0204_L3.6mm_D1.6mm_P5.08mm_Horizontal; LCSC C11702 -> (none)
Connections:
- net IO15: no longer names the net of U1.8 (IO15)
- net IO16: no longer names the net of U1.9 (IO16)
- net IO18: no longer names the net of U1.11 (IO18)
- net IO19: no longer names the net of U1.13 (IO19)
- net IO20: no longer names the net of U1.14 (IO20)
- net IO21: no longer names the net of U1.23 (IO21)
- net IO35: no longer names the net of U1.28 (IO35)
- net IO36: no longer names the net of U1.29 (IO36)
- net IO37: no longer names the net of U1.30 (IO37)
- no-connect marks 22 -> 31
